File: Hardware/Top/Smarty-TOP.sch (EAGLE design)
At the start: 52 parts, among them SW6 SWITCH.MOM, SW7 SWITCH.MOM, SW8 SWITCH.MOM, U2 NRF52832_MODULE_MDBT42, U4 PCF8523

Commit message: Take 001 and part of Take 002 Completed
Parts:
- removed C10, C11: 300p, LinnesLab-Passives:CAPACITOR0603
- removed C12: 10u, LinnesLab-Passives:CAPACITOR0805
- removed C14: 100n, LinnesLab-Passives:CAPACITOR0603
- removed CORTEX1: CORTEX_DEBUG_PTH, LinnesLab-Connectors:CORTEX_DEBUG_PTH
- removed D1: (no value), LinnesLab-DiscreteSemi:SCHOTTKY-USC
- removed L2: 10u, LinnesLab-Passives:INDUCTOR0603
- removed R8, R9: 10k, LinnesLab-Passives:RESISTOR0603
- removed SW3, SW4: (no value), LinnesLab-Switches:SPST-PTS830GG140-COPY.1-3
- removed XTAL2: 32.768kHz, LinnesLab-Clocks:CRYSTALECS-.327-12.5-12-C-TR
- added C26: 1u, LinnesLab-Passives:CAPACITOR0603
- added C27, C28: (no value), LinnesLab-Passives:CAPACITOR0603
- added C29, C30: 300p, LinnesLab-Passives:CAPACITOR0603
- added C31: 10u, LinnesLab-Passives:CAPACITOR0805
- added C32: 100n, LinnesLab-Passives:CAPACITOR0603
- added CORTEX3: CORTEX_DEBUG_PTH, LinnesLab-Connectors:CORTEX_DEBUG_PTH
- added D3: (no value), LinnesLab-DiscreteSemi:SCHOTTKY-USC
- added JP2: (no value), LinnesLab-Switches:JUMPER-SMT_2_NO_SILK
- added L3: 10u, LinnesLab-Passives:INDUCTOR0603
- added LED5: RED, LinnesLab-LED:LED0603
- added LED6: BLUE, LinnesLab-LED:LED0603
- added R1, R2: 0, LinnesLab-Passives:RESISTOR0603
- added R10: 27, LinnesLab-Passives:RESISTOR0603
- added R16, R17, R19, R20: 1k, LinnesLab-Passives:RESISTOR0603
- added R18: 10k, LinnesLab-Passives:RESISTOR0603
- added SW1: SWITCH.MOM, LinnesLab-Switches:SWITCH.MOM
- added U5: NRF52832_MODULE_MDBT42, LinnesLab-Microcontrollers:NRF52832_MODULE_MDBT42
- added XTAL4: 32.768kHz, LinnesLab-Clocks:CRYSTALECS-.327-12.5-12-C-TR
- C7: value 1u -> 100n
- C8, C9: value (none) -> 47p
- LED4: value BLUE -> YELLOW
- R3, R4: value 1k -> 10k
- R5: value 10k -> 27
- SW7, SW8: value SWITCH.MOM -> (none); device LinnesLab-Switches:SWITCH.MOM -> LinnesLab-Switches:SPST-PTS830GG140-COPY.1-3
- U2: value NRF52832_MODULE_MDBT42 -> FT231XS; device LinnesLab-Microcontrollers:NRF52832_MODULE_MDBT42 -> LinnesLab-DigitalIC:FT231XS
- XTAL3: FREQ 32.7680KHZ -> (none)
Connections:
- removed net N$10: LED4.A, R4.1
- removed net N$18: SW6.3, SW6.4
- removed net N$21: SW7.1, SW7.2
- removed net N$22: SW7.3, SW7.4
- removed net N$23: SW8.1, SW8.2
- removed net N$24: SW8.3, SW8.4
- removed net N$4: C8.2, U2.P0.00/XL1, XTAL2.1
- removed net N$6: C9.1, U2.P0.01/XL2, XTAL2.2
- removed net N$9: LED3.A, R3.1
- removed net RXD: U2.P0.08
- removed net TXD: U2.P0.06
- removed net VBATT: U4.VBAT
- new net !CTS: JP2.2, U2.!CTS
- new net FT3V3: U2.3V3OUT
- new net N$26: C27.2, U5.P0.00/XL1, XTAL4.1
- new net N$27: C28.1, U5.P0.01/XL2, XTAL4.2
- new net N$28: LED5.A, R16.1
- new net N$29: LED6.A, R17.1
- new net N$30: L3.1, U5.DCC
- new net N$31: C26.1, L3.2, U5.DEC4
- new net N$32: CORTEX3.NC/TDI
- new net RXD.FT: R2.1, U2.RXD
- new net RXD.NRF: R1.2, U5.P0.08
- new net RXLED: R19.1, U2.CBUS1
- new net SW1: SW1.1, SW6.1
- new net TXD.FT: R1.1, U2.TXD
- new net TXD.NRF: R2.2, U5.P0.06
- new net TXLED: R20.1, U2.CBUS2
- net 3.3V: now also C31.2, C7.2, CORTEX3.VCC, D3.C, LED3.A, LED4.A, R18.2, R3.2, R4.2, U2.!RESET, U2.VCCIO, U5.VDD; no longer C12.2, CORTEX1.VCC, D1.C, R5.2, R8.2, R9.2, U2.VDD
- net DFU: now also SW7.B, U5.P0.20; no longer SW3.B, U2.P0.20
- net DTR: now also C32.1, U2.!DTR; no longer C14.1
- net FRST: now also U5.P0.22; no longer U2.P0.22
- net GND: now also C26.2, C27.1, C28.2, C29.2, C30.2, C31.1, C7.1, C8.2, C9.1, CORTEX3.GND@3, CORTEX3.GND@5, CORTEX3.GNDDTCT, CORTEX3.KEY, JP2.1, LED5.C, LED6.C, SW1.3, SW1.4, SW6.3, SW6.4, SW7.A, SW8.B, U2.GND@16, U2.GND@6, U5.GND@1, U5.GND@2, U5.GND@3, U5.GND@4, USB2.SHIELD; no longer C10.2, C11.2, C12.1, C7.2, C8.1, C9.2, CORTEX1.GND@3, CORTEX1.GND@5, CORTEX1.GNDDTCT, CORTEX1.KEY, LED3.C, LED4.C, SW3.A, SW4.B, U2.GND@1, U2.GND@2, U2.GND@3, U2.GND@4
- net LED1: now also R16.2, U5.P0.17; no longer R3.2, U2.P0.17
- net LED2: now also R17.2, U5.P0.19; no longer R4.2, U2.P0.19
- net MISO: now also U5.P0.14; no longer U2.P0.14
- net MOSI: now also U5.P0.13; no longer U2.P0.13
- net N$11: now also R5.2, U2.USBDM; no longer L2.1, U2.DCC
- net N$12: now also R10.2, U2.USBDP; no longer C7.1, L2.2, U2.DEC4
- net N$14: now also LED3.C, R19.2; no longer CORTEX1.NC/TDI
- net N$16: now also LED4.C, R20.2; no longer SW6.1, SW6.2
- net P0.09/NFC1: now also C30.1, U5.P0.09; no longer C11.1, U2.P0.09
- net P0.10/NFC2: now also C29.1, U5.P0.10; no longer C10.1, U2.P0.10
- net RESET: now also C32.2, CORTEX3.!RESET, D3.A, R18.1, SW8.A, U5.P0.21/RESET; no longer C14.2, CORTEX1.!RESET, D1.A, R5.1, SW4.A, U2.P0.21/RESET
- net SCK: now also U5.P0.12; no longer U2.P0.12
- net SCL: now also R4.1, U5.P0.26; no longer R8.1, U2.P0.26
- net SDA: now also R3.1, U5.P0.25; no longer R9.1, U2.P0.25
- net SWCLK: now also CORTEX3.SWDCLK/TCK, U5.SWDCLK; no longer CORTEX1.SWDCLK/TCK, U2.SWDCLK
- net SWDIO: now also CORTEX3.SWDIO/TMS, U5.SWDIO; no longer CORTEX1.SWDIO/TMS, U2.SWDIO
- net SWO: now also CORTEX3.SWO/TDO, U5.P0.18/SWO; no longer CORTEX1.SWO/TDO, U2.P0.18/SWO
- net USB+: now also C8.1, R10.1
- net USB-: now also C9.2, R5.1
- net V_USB: now also U2.VCC
Other:
- note added: "Additional notes for advanced users only"
- note added: "Digital Outputs CS.OLED RESET.OLED DC.OLED [SPI] [I2C] SD.CS (Optional) Card Detect 1 and 2 Digital Inputs 3x buttons Charge Status Analog Inputs Battery Monitor Analog Outputs"
- note added: "FTDI Serial-to-USB Converter"
- note added: "I don't remember if CTS needs to be grounded or left floating so here's a jumper to ground so it can be configued either way dynamically."
- note added: "Notes"
- note added: "PIN_DFU / P0.20: If this pin is detected to be at GND level at startup, the board will enter a special serial bootloader mode and will not execute any user code, going straight into bootloader mode. If you wish to use this pin as a standard GPIO, make sure that it is pulled high with a pullup resistor so that your code will execute normally when the MCU starts up. FRST/P0.22: Setting this pin to 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"
- note added: "SPECIAL / PORT / PIN ON PACKAGE / GPIO(D_or_A) / Comments Factory Reset / P0.22 / pin38 / DO NOT USE FOR ANY GPIO SWDIO / none / pin37 / reserved-not available for general GPIO SWCLK / none / pin36 / reserved-not available for general GPIO RESET / P0.21 / pin35 / reserved-not available for general GPIO DFU / P0.20 / pin34 / reserved-not available for general GPIO LED2 / P0.19 / pin33 / reserved f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"
- note added: "SPECIAL / PORT / PIN ON PACKAGE / GPIO(D_or_A) / Comments SDA / P0.25 / pin2 / D25 SCL / P0.26 / pin3 / D26 none / P0.27 / pin4 / D27 none / P0.28 / pin5 / D28_or_A4 / (low drive, low frequency IO) none / P0.29 / pin6 / D29_or_A5 / (low drive, low frequency IO) none / P0.30 / pin7 / D30_or_A6 none / P0.31 / pin8 / D31_or_A7 / (Battery monitoring on Adafruit boards)"
- note added: "SPECIAL / PORT / PIN ON PACKAGE / GPIO(D_or_A) / Comments none / P0.02 / pin15 / D2_or_A0 none / P0.03 / pin16 / D3_or_A1 none / P0.04 / pin17 / D4_or_A2 none / P0.05 / pin18 / D5_or_A3 TXD / P0.06 / pin19 / D6 / but reserved for Serial communication and programming none / P0.07 / pin20 / D7 RXD / P0.08 / pin21 / D8 / but reserved for Serial communication and programming NFC1 / P0.09 / pin22 / D9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"
- note added: "Some pins are noted as reserved and not available for general GPIO (unless you are an adavanced user) I2C, SPI, and SWD pins can be repurposed if you know what you are doing For Milestones, avoid repurposing NFC pins. For P0.19 (LED2), Adafruit's Bluetooth Low Energy libraries use this pin to indicated successful pairing. The LED blinks when the device is doing some Bluetooth process and stays li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"
- note added: "TXD goes to RX on the other device RXD goes to TX on the other device"
- note removed: "Back-up battery if desired"
- moved on the sheet: C2, C7, C8, C9, LED3, LED4, R3, R4, R5, SD2, SW6, U4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

Commit message: Finished Take 2
Parts:
- removed SW6: SWITCH.MOM, LinnesLab-Switches:SWITCH.MOM
- added J1: (no value), LinnesLab-Connectors:CONN_07
- added SW2: SWITCH.MOM, LinnesLab-Switches:SWITCH.MOM
Connections:
- removed net BATT: R13.1, R14.2
- removed net CD1: SD2.CARD_DETECT
- removed net CHRG.STAT: CHRG2.STAT, R12.1
- removed net CS.OLED: U3./CS
- removed net DC.OLED: U3.DC/I2C_SA0
- removed net RESET.OLED: U3./RES
- removed net SD.CS: SD2.CS
- removed net SW1: SW1.1, SW6.1
- new net A4/BATT: R13.1, R14.2, U5.P0.28/AIN4
- new net A6/TIA: U5.P0.30/AIN6
- new net A7/PPG: U5.P0.31/AIN7
- new net D11/SW1: SW1.1, U5.P0.11
- new net D15/SW2: SW2.1, U5.P0.15
- new net D16/CS.OLED: U3./CS, U5.P0.16
- new net D27/CHRG.STATUS: CHRG2.STAT, R12.1, U5.P0.27
- new net D29/LED.CTRL: U5.P0.29/AIN5
- new net D3/RESET.OLED: U3./RES, U5.P0.03/AIN1
- new net D4/DC.OLED: U3.DC/I2C_SA0, U5.P0.04/AIN2
- new net D5/CD1: SD2.CARD_DETECT, U5.P0.05/AIN3
- new net D7/SD.CS: SD2.CS, U5.P0.07
- net GND: now also SW2.3, SW2.4; no longer SW6.3, SW6.4
Other:
- note added: "Digital Output"
- moved on the sheet: R3, R4, SW1, SW7, SW8

Commit message: Finished Take 004
Parts:
- removed J1: (no value), LinnesLab-Connectors:CONN_07
- removed R15: 100k, LinnesLab-Passives:RESISTOR0603
- added J3: (no value), LinnesLab-Connectors:CONN_07-1.27MM
- renumbered CHRG2 to CHRG, LDO2 to LDO1
Connections:
- net 3.3V: now also J3.4; no longer R15.2
- net A6/TIA: now also J3.6
- net A7/PPG: now also J3.7
- net D29/LED.CTRL: now also J3.5
- net GND: now also J3.3; no longer R15.1, SW1.4, SW2.4
- net SCL: now also J3.2
- net SDA: now also J3.1
Other:
- note added: "Connection to Bottom Board"

Commit message: Finished Take 006
Parts:
- removed C2, C5, C6: 1u, LinnesLab-Passives:CAPACITOR0603
- removed C20, C21: 4.7u, LinnesLab-Passives:CAPACITOR0603
- removed CHRG: MCP73831, LinnesLab-Power:MCP73831
- removed LDO1: MIC5504, LinnesLab-Power:MIC5504
- removed R11: (no value), LinnesLab-Passives:RESISTOR0603
- removed R12: 100k, LinnesLab-Passives:RESISTOR0603
- removed SD2: (no value), LinnesLab-Connectors:MICROSD
- removed U4: PCF8523, LinnesLab-Clocks:PCF8523
- removed XTAL3: 32.7680kHz, LinnesLab-Clocks:CRYSTALECS-.327-12.5-12-C-TR
Connections:
- removed net CD2: SD2.CARD_DETECT1
- removed net N$17: CHRG.PROG, R11.2
- removed net N$19: U4.OSCO, XTAL3.1
- removed net N$20: U4.OSCI, XTAL3.2
- net 3.3V: no longer C2.1, C6.1, LDO1.OUT, SD2.VDD, U4.VDD
- net D27/CHRG.STATUS: no longer CHRG.STAT, R12.1
- net D5/CD1: no longer SD2.CARD_DETECT
- net D7/SD.CS: no longer SD2.CS
- net GND: no longer C2.2, C20.2, C21.1, C5.1, C6.2, CHRG.VSS, LDO1.GND, R11.1, SD2.GND, SD2.GND1, SD2.VSS, U4.VSS
- net MISO: no longer SD2.DATA_OUT
- net MOSI: no longer SD2.DATA_IN
- net SCK: no longer SD2.SCLK
- net SCL: no longer U4.SCL
- net SDA: no longer U4.SDA
- net VIN: no longer C21.2, C5.2, CHRG.VIN, LDO1.EN, LDO1.IN, R12.2
- net VLIPO: no longer C20.1, CHRG.VBAT
Other:
- note removed: "Connect MISO, MOSI, and SCK to appropriate pins on microcontroller. Those are SPI pins and are generally prespecified. You have more flexibility with the SD.CS pin."
- note removed: "Digital Output"
- note removed: "I2C Address = 0x68h"
- note removed: "Real-Time Clock"
- note removed: "SD Card"

Commit message: Almost Done With Take 008
Parts:
- removed C19: 2.2uF, LinnesLab-Passives:CAPACITOR0402
- removed C29, C30: 300p, LinnesLab-Passives:CAPACITOR0603
- removed C32: 100n, LinnesLab-Passives:CAPACITOR0603
- removed CORTEX3: CORTEX_DEBUG_PTH, LinnesLab-Connectors:CORTEX_DEBUG_PTH
- removed D4, D5: (no value), LinnesLab-DiscreteSemi:SCHOTTKY-USC
- removed J3: (no value), LinnesLab-Connectors:CONN_07-1.27MM
- removed R18: 10k, LinnesLab-Passives:RESISTOR0603
- removed R19: 1k, LinnesLab-Passives:RESISTOR0603
- removed SW7, SW8: (no value), LinnesLab-Switches:SPST-PTS830GG140-COPY.1-3
- removed USB2: USB.MICRO-BIGGERPADS, LinnesLab-Connectors:USB.MICRO-BIGGERPADS
- added C10, C12: 100n, LinnesLab-Passives:CAPACITOR0603
- added C11: 47p, LinnesLab-Passives:CAPACITOR0603
- added C14: 2.2uF, LinnesLab-Passives:CAPACITOR0402
- added C5: 4.7u, LinnesLab-Passives:CAPACITOR0603
- added C6: 1u, LinnesLab-Passives:CAPACITOR0603
- added CHRG1: MCP73831, LinnesLab-Power:MCP73831
- added D1, D2: (no value), LinnesLab-DiscreteSemi:SCHOTTKY-USC
- added DEBUG1: CORTEX_DEBUG_PTH, LinnesLab-Connectors:CORTEX_DEBUG_PTH
- added J1: (no value), LinnesLab-Connectors:CONN_07-1.27MM
- added LDO1: MIC5504, LinnesLab-Power:MIC5504
- added R11: 27, LinnesLab-Passives:RESISTOR0603
- added R12, R9: 10k, LinnesLab-Passives:RESISTOR0603
- added R8: 100k, LinnesLab-Passives:RESISTOR0603
- added RESET: (no value), LinnesLab-Switches:SPST-PTS830GG140-COPY.1-3
- added SW3: SWITCH.MOM, LinnesLab-Switches:SWITCH.MOM
- added USB1: USB.MICRO-BIGGERPADS, LinnesLab-Connectors:USB.MICRO-BIGGERPADS
- C13: value 2.2uF -> 10uF; device LinnesLab-Passives:CAPACITOR0402 -> LinnesLab-Passives:CAPACITOR0603
- C15: device LinnesLab-Passives:CAPACITOR0402 -> LinnesLab-Passives:CAPACITOR0603
- C16: value 10uF -> 2.2uF; device LinnesLab-Passives:CAPACITOR0603 -> LinnesLab-Passives:CAPACITOR0402
- C7: value 100n -> 1u
- C8: value 47p -> 4.7u
- R1, R2: value 0 -> 10k
- R13: value 100k -> 390k
- R14: value 100k -> 1k
- R16, R17: value 1k -> 0
- R3: value 10k -> 100k
- R4: value 10k -> 1k
- R5: value 27 -> 1k
- R6: value 10k -> (none)
- R7: value 390k -> 100k
- SW2: value SWITCH.MOM -> (none); device LinnesLab-Switches:SWITCH.MOM -> LinnesLab-Switches:SPST-PTS830GG140-COPY.1-3
- renumbered C26 to C1, C27 to C3, C28 to C4, C31 to C2, JP2 to JP1, L3 to L1, LED5 to LED1, LED6 to LED2, R20 to R15, U5 to U1, XTAL4 to XTAL1
Connections:
- removed net A4/BATT: R13.1, R14.2, U1.P0.28/AIN4
- removed net A6/TIA: J3.6, U1.P0.30/AIN6
- removed net A7/PPG: J3.7, U1.P0.31/AIN7
- removed net D29/LED.CTRL: J3.5, U1.P0.29/AIN5
- new net A4/PPG: J1.7, U1.P0.28/AIN4
- new net A5/TIA: J1.6, U1.P0.29/AIN5
- new net A7/BATT: R7.1, R8.2, U1.P0.31/AIN7
- new net D30/LED.CTRL: J1.5, U1.P0.30/AIN6
- new net N$4: CHRG1.PROG, R6.2
- net 3.3V: now also C12.2, C18.2, C7.1, DEBUG1.VCC, J1.4, LDO1.OUT, R1.2, R2.2, R9.2; no longer C19.2, C7.2, CORTEX3.VCC, J3.4, R18.2, R3.2, R4.2
- net D15/SW2: now also SW3.1; no longer SW2.1
- net D27/CHRG.STATUS: now also CHRG1.STAT, R3.1
- net DFU: now also SW2.B; no longer SW7.B
- net DTR: now also C10.1; no longer C32.1
- net GND: now also C11.2, C12.1, C13.1, C15.1, C5.1, C6.1, C7.2, CHRG1.VSS, DEBUG1.GND@3, DEBUG1.GND@5, DEBUG1.GNDDTCT, DEBUG1.KEY, J1.3, LDO1.GND, R12.1, R13.2, R8.1, RESET.B, SW2.A, SW3.3, USB1.GND, USB1.SHIELD; no longer C16.1, C19.1, C29.2, C30.2, C7.1, CORTEX3.GND@3, CORTEX3.GND@5, CORTEX3.GNDDTCT, CORTEX3.KEY, J3.3, R14.1, R7.2, SW2.3, SW7.A, SW8.B, USB2.GND, USB2.SHIELD
- net LED1: now also R4.2; no longer R16.2
- net LED2: now also R5.2; no longer R17.2
- net N$1: now also R12.2; no longer R6.2
- net N$11: now also R10.2; no longer R5.2
- net N$12: now also R11.2; no longer R10.2
- net N$13: now also C13.2; no longer C16.2
- net N$14: now also R14.2; no longer R19.2
- net N$15: now also C15.2; no longer C18.2
- net N$2: now also R13.1; no longer R7.1
- net N$28: now also R4.1; no longer R16.1
- net N$29: now also R5.1; no longer R17.1
- net N$3: now also C16.2; no longer C13.2
- net N$32: now also DEBUG1.NC/TDI; no longer CORTEX3.NC/TDI
- net N$5: now also C16.1; no longer C13.1
- net N$7: now also C14.2; no longer C15.2
- net N$8: now also C14.1; no longer C15.1
- net P0.09/NFC1: no longer C30.1
- net P0.10/NFC2: no longer C29.1
- net RESET: now also C10.2, DEBUG1.!RESET, R9.1, RESET.A; no longer C32.2, CORTEX3.!RESET, R18.1, SW8.A
- net RXD.FT: now also R17.1; no longer R2.1
- net RXD.NRF: now also R16.2; no longer R1.2
- net RXLED: now also R14.1; no longer R19.1
- net SCL: now also J1.2, R2.1; no longer J3.2, R4.1
- net SDA: now also J1.1, R1.1; no longer J3.1, R3.1
- net SWCLK: now also DEBUG1.SWDCLK/TCK; no longer CORTEX3.SWDCLK/TCK
- net SWDIO: now also DEBUG1.SWDIO/TMS; no longer CORTEX3.SWDIO/TMS
- net SWO: now also DEBUG1.SWO/TDO; no longer CORTEX3.SWO/TDO
- net TXD.FT: now also R16.1; no longer R1.1
- net TXD.NRF: now also R17.2; no longer R2.2
- net USB+: now also C11.1, R11.1, USB1.D+; no longer C8.1, R10.1, USB2.D+
- net USB-: now also R10.1, USB1.D-; no longer R5.1, USB2.D-
- net VIN: now also C5.2, C6.2, CHRG1.VIN, D1.C, D2.C, LDO1.EN, LDO1.IN, R3.2; no longer D4.C, D5.C
- net VLIPO: now also C8.1, CHRG1.VBAT, D1.A, R7.2; no longer D4.A, R13.2
- net V_USB: now also D2.A, USB1.V+; no longer D5.A, USB2.V+
Other:
- note added: "Bottom Board Connection"
- note added: "Digital Output"
- note added: "Diodes switch from Lipo Power to USB when USB is connected. The USB Power then charges the battery."
- note added: "Notes: Smarty Basic Top- Revision A Date: July 2, 2020 Author: Julia Talor"
- note added: "R11 sets charge current I_charge = 1000V / R11 per MCP73831 datasheet"
- note added: "Voltage Division used to monitor battery voltage."
- note removed: "Connection to Bottom Board"
- note removed: "Digital Outputs CS.OLED RESET.OLED DC.OLED [SPI] [I2C] SD.CS (Optional) Card Detect 1 and 2 Digital Inputs 3x buttons Charge Status Analog Inputs Battery Monitor Analog Outputs"
- note removed: "Notes"
- moved on the sheet: C13, C15, C16, C17, C18, C7, C8, D3, J2, R1, R10, R13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
