File: Hardware/Bottom/Smarty-BOTTOM.brd (EAGLE design)
At the start: 160 x 100 mm, 0 parts

Commit message: Take 001 and part of Take 002 Completed
Parts:
- added C1, C10, C11, C17, C18, C22: 100n, LinnesLab-Passives:C0603
- added C14, C19: 2.2n, LinnesLab-Passives:C0603
- added C15, C16: 2.2u, LinnesLab-Passives:C0603
- added C20: 22u, LinnesLab-Passives:C0603
- added C21: 22n, LinnesLab-Passives:C0603
- added IMU1: LSM6DS3_CAST, LinnesLab-Sensors:LSM6DS3_CAST
- added OP3: (no value), LinnesLab-AnalogIC:SO14
- added OP4: (no value), LinnesLab-AnalogIC:SOT23-5
- added Q1: (no value), LinnesLab-DiscreteSemi:SOT23-3
- added R13, R15, R19, R21: 220k, LinnesLab-Passives:R0603
- added R14, R22: 10M, LinnesLab-Passives:R0603
- added R16: (no value), LinnesLab-Passives:R0603
- added R17, R18: 10k, LinnesLab-Passives:R0402
- added R20, R23: 1M, LinnesLab-Passives:R0603
- added R24: 10k, LinnesLab-Passives:R0603
- added U$3: (no value), LinnesLab-Connectors:PPG.MODULE.2
- added U$4: AD5171, LinnesLab-DigitalIC:SOT-23-8
- added U1: AD5242-SO16, LinnesLab-DigitalIC:SO16
Connections:
- new net 3.3V: C1.2, C11.2, C17.2, C18.2, C22.2, IMU1.2, OP3.4, OP4.5, R13.2, R15.2, R17.2, U$3.V+, U$4.2, U$4.6, U1.5, U1.6
- new net G.A1: U1.2
- new net G.A2: U1.16
- new net G.O1: U1.1
- new net G.O2: U1.13
- new net G.W2: C21.1, OP3.2, R24.1, U1.15
- new net GND: C1.1, C11.1, C17.1, C18.1, C22.1, IMU1.1, OP3.11, OP4.2, OP4.3, Q1.2, R18.1, R19.1, R21.1, U$3.GND, U$4.3, U1.10, U1.11, U1.12, U1.9
- new net LED: Q1.3
- new net LED.C: U$3.LD1
- new net LED.CTRL: U$4.8
- new net N$10: OP3.12, R17.1, R18.2
- new net N$13: C15.2, OP3.5, R13.1, R19.2
- new net N$15: C14.2, OP3.6, R14.1, R20.2
- new net N$16: C14.1, C16.1, OP3.7, R14.2
- new net N$17: C16.2, OP3.10, R15.1, R21.2
- new net N$18: C19.2, OP3.9, R22.1, R23.2
- new net N$19: C19.1, C20.1, OP3.8, R22.2
- new net N$20: C20.2, R24.2
- new net N$8: Q1.1, R16.2
- new net N$9: R16.1, U$4.1, U$4.7
- new net PD.C: C10.1, OP4.4, U$3.PD, U1.4
- new net PPG: C21.2, OP3.1, U1.14
- new net SCL: IMU1.3, U$4.4, U1.7
- new net SDA: IMU1.4, U$4.5, U1.8
- new net TIA: C10.2, C15.1, OP4.1, U1.3
- new net VREF: OP3.13, OP3.14, OP3.3, R20.1, R23.1
Routing:
- added copper zone on layer 1, net 3.3V
Other:
- board size 160 x 100 mm -> 33 x 33 mm

Commit message: Finished Take 2
Parts:
- added J1: (no value), LinnesLab-Connectors:1X07
- moved C15 3.36 mm to (21.9, 29.8)
- moved C10 3.09 mm to (24.4, 29.8)
- moved R19 1.73 mm to (6.05, 30.0)
- moved R17 1.02 mm to (11.8, 30.2)
Connections:
- removed net LED.CTRL: U$4.8
- removed net PPG: C21.2, OP3.1, U1.14
- removed net TIA: C10.2, C15.1, OP4.1, U1.3
- new net A6/TIA: C10.2, C15.1, J1.5, OP4.1, U1.3
- new net A7/PPG: C21.2, J1.7, OP3.1, U1.14
- new net D29/LED.CTRL: J1.6, U$4.8
Changed lines of the file:
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@@
 <setting verticaltext="up"/>
 </settings>
-<grid distance="1" unitdist="mil" unit="mil" style="lines" multiple="1" display="no" altdistance="5" altunitdist="mil" altunit="mil"/>
+<grid distance="1" unitdist="mil" unit="mm" style="lines" multiple="1" display="no" altdistance="5" altunitdist="mil" altunit="mil"/>
 <layers>
 <layer number="1" name="Top" color="4" fill="1" visible="yes" active="yes"/>
@@
 <elements>
 <element name="U$3" library="LinnesLab-Connectors" package="PPG.MODULE.2" value="" x="19" y="19" locked="yes" smashed="yes"/>
-<element name="C10" library="LinnesLab-Passives" package="C0603" value="100n" x="23.9014" y="32.8676" smashed="yes" rot="R90">
-<attribute name="NAME" x="23.2664" y="32.2326" size="0.6604" layer="25" rot="R90"/>
-<attribute name="VALUE" x="25.8064" y="32.2326" size="1.27" layer="27" rot="R90"/>
+<element name="C10" library="LinnesLab-Passives" package="C0603" value="100n" x="24.384" y="29.8196" smashed="yes" rot="R90">
+<attribute name="NAME" x="23.749" y="29.1846" size="0.6604" layer="25" rot="R90"/>
+<attribute name="VALUE" x="26.289" y="29.1846" size="1.27" layer="27" rot="R90"/>
 </element>
 <element name="C11" library="LinnesLab-Passives" package="C0603" value="100n" x="18.5166" y="29.0576" smashed="yes">
@@
 <attribute name="VALUE" x="19.7866" y="25.9588" size="1.27" layer="27" rot="R90"/>
 </element>
-<element name="C15" library="LinnesLab-Passives" package="C0603" value="2.2u" x="21.1836" y="33.0454" smashed="yes" rot="R270">
-<attribute name="NAME" x="21.8186" y="33.6804" size="0.6604" layer="25" rot="R270"/>
-<attribute name="VALUE" x="19.2786" y="33.6804" size="1.27" layer="27" rot="R270"/>
+<element name="C15" library="LinnesLab-Passives" package="C0603" value="2.2u" x="21.9202" y="29.7688" smashed="yes" rot="R270">
+<attribute name="NAME" x="22.5552" y="30.4038" size="0.6604" layer="25" rot="R270"/>
+<attribute name="VALUE" x="20.0152" y="30.4038" size="1.27" layer="27" rot="R270"/>
 </element>
 <element name="C16" library="LinnesLab-Passives" package="C0603" value="2.2u" x="26.8732" y="21.9202" smashed="yes">
@@
 <attribute name="VALUE" x="27.2288" y="22.4282" size="1.27" layer="27"/>
 </element>
-<element name="R17" library="LinnesLab-Passives" package="R0402" package3d_urn="urn:adsk.eagle:package:15661898/2" value="10k" x="11.7094" y="31.2166" smashed="yes">
-<attribute name="NAME" x="11.0744" y="31.8516" size="1.27" layer="25"/>
-<attribute name="VALUE" x="11.0744" y="29.3116" size="1.27" layer="27"/>
+<element name="R17" library="LinnesLab-Passives" package="R0402" package3d_urn="urn:adsk.eagle:package:15661898/2" value="10k" x="11.811" y="30.2006" smashed="yes">
+<attribute name="NAME" x="11.176" y="30.8356" size="1.27" layer="25"/>
+<attribute name="VALUE" x="11.176" y="28.2956" size="1.27" layer="27"/>
 </element>
 <element name="R18" library="LinnesLab-Passives" package="R0402" package3d_urn="urn:adsk.eagle:package:15661898/2" value="10k" x="11.7094" y="27.7368" smashed="yes">
@@
 <attribute name="VALUE" x="27.7622" y="14.5542" size="1.27" layer="27" ratio="10" rot="R270"/>
 </element>
-<element name="R19" library="LinnesLab-Passives" package="R0603" package3d_urn="urn:adsk.eagle:package:15661944/2" value="220k" x="5.969" y="31.6992" smashed="yes">
-<attribute name="NAME" x="5.334" y="32.3342" size="1.27" layer="25"/>
-<attribute name="VALUE" x="5.334" y="29.7942" size="1.27" layer="27"/>
+<element name="R19" library="LinnesLab-Passives" package="R0603" package3d_urn="urn:adsk.eagle:package:15661944/2" value="220k" x="6.0452" y="29.972" smashed="yes">
+<attribute name="NAME" x="5.4102" y="30.607" size="1.27" layer="25"/>
+<attribute name="VALUE" x="5.4102" y="28.067" size="1.27" layer="27"/>
 </element>
 <element name="R20" library="LinnesLab-Passives" package="R0603" package3d_urn="urn:adsk.eagle:package:15661944/2" value="1M" x="5.969" y="26.8224" smashed="yes">
@@
 <attribute name="NAME" x="6.0198" y="7.0104" size="0.6604" layer="25" rot="R270"/>
 <attribute name="VALUE" x="3.4798" y="7.0104" size="0.6604" layer="27" rot="R270"/>
+</element>
+<element name="J1" library="LinnesLab-Connectors" package="1X07" value="" x="5" y="33" smashed="yes">
+<attribute name="NAME" x="3.73" y="34.397" size="0.6096" layer="25" font="vector" ratio="20"/>
+<attribute name="VALUE" x="3.73" y="30.968" size="0.6096" layer="27" font="vector" ratio="20"/>
 </element>
 </elements>
@@
 <wire x1="19.6444" y1="14.8242" x2="16.5146" y2="11.549" width="0" layer="19" extent="1-1"/>
 <wire x1="5.2206" y1="21.5392" x2="11.2404" y2="19.4056" width="0" layer="19" extent="1-1"/>
-<wire x1="5.119" y1="31.6992" x2="11.0594" y2="27.7368" width="0" layer="19" extent="1-1"/>
+<wire x1="5.1952" y1="29.972" x2="11.0594" y2="27.7368" width="0" layer="19" extent="1-1"/>
 <wire x1="11.4182" y1="6.2992" x2="16.5146" y2="11.549" width="0" layer="19" extent="1-1"/>
 <wire x1="7.5438" y1="7.8994" x2="11.4182" y2="6.2992" width="0" layer="19" extent="1-1"/>
@@
 <wire x1="12.6238" y1="5.3594" x2="17.1646" y2="11.549" width="0" layer="19" extent="1-1"/>
 </signal>
-<signal name="TIA">
+<signal name="A6/TIA">
 <contactref element="C10" pad="2"/>
 <contactref element="U1" pad="3"/>
 <contactref element="C15" pad="1"/>
 <contactref element="OP4" pad="1"/>
-<wire x1="21.1836" y1="33.8954" x2="23.9014" y2="33.7176" width="0" layer="19" extent="1-1"/>
-<wire x1="12.5882" y1="25.3132" x2="21.1836" y2="33.8954" width="0" layer="19" extent="1-1"/>
+<contactref element="J1" pad="5"/>
+<wire x1="21.9202" y1="30.6188" x2="24.384" y2="30.6696" width="0" layer="19" extent="1-1"/>
+<wire x1="15.16" y1="33" x2="21.9202" y2="30.6188" width="0" layer="19" extent="1-1"/>
+<wire x1="12.5882" y1="25.3132" x2="15.16" y2="33" width="0" layer="19" extent="1-1"/>
 <wire x1="25.3238" y1="12.3952" x2="12.5882" y2="25.3132" width="0" layer="19" extent="1-1"/>
 </signal>
@@
 <contactref element="U1" pad="4"/>
 <contactref element="OP4" pad="4"/>
-<wire x1="17.73" y1="24.08" x2="23.9014" y2="32.0176" width="0" layer="19" extent="1-1"/>
+<wire x1="17.73" y1="24.08" x2="24.384" y2="28.9696" width="0" layer="19" extent="1-1"/>
 <wire x1="14.4882" y1="27.9252" x2="17.73" y2="24.08" width="0" layer="19" extent="1-1"/>
 <wire x1="25.3238" y1="11.1252" x2="17.73" y2="24.08" width="0" layer="19" extent="1-1"/>
@@
 <wire x1="10.4022" y1="11.7348" x2="15.2146" y2="11.549" width="0" layer="19" extent="1-1"/>
 </signal>
-<signal name="LED.CTRL">
+<signal name="D29/LED.CTRL">
 <contactref element="U$4" pad="8"/>
+<contactref element="J1" pad="6"/>
+<wire x1="15.2146" y1="13.9018" x2="17.7" y2="33" width="0" layer="19" extent="1-1"/>
 </signal>
 <signal name="N$10">
@@
 <contactref element="R18" pad="2"/>
 <wire x1="12.3594" y1="27.7368" x2="31.7338" y2="29.5402" width="0" layer="19" extent="1-1"/>
-<wire x1="11.0594" y1="31.2166" x2="12.3594" y2="27.7368" width="0" layer="19" extent="1-1"/>
+<wire x1="11.161" y1="30.2006" x2="12.3594" y2="27.7368" width="0" layer="19" extent="1-1"/>
 </signal>
 <signal name="LED">
@@
 <contactref element="U1" pad="1"/>
 </signal>
-<signal name="PPG">
+<signal name="A7/PPG">
 <contactref element="U1" pad="14"/>
 <contactref element="C21" pad="2"/>
 <contactref element="OP3" pad="1"/>
+<contactref element="J1" pad="7"/>
+<wire x1="20.24" y1="33" x2="26.5338" y2="32.0802" width="0" layer="19" extent="1-1"/>
 <wire x1="31.4706" y1="12.3952" x2="26.5338" y2="32.0802" width="0" layer="19" extent="1-1"/>
 <wire x1="13.1182" y1="11.3792" x2="31.4706" y2="12.3952" width="0" layer="19" extent="1-1"/>
@@
 <contactref element="R19" pad="2"/>
 <contactref element="OP3" pad="5"/>
-<wire x1="17.7428" y1="30.5308" x2="21.1836" y2="32.1954" width="0" layer="19" extent="1-1"/>
-<wire x1="26.5338" y1="27.0002" x2="21.1836" y2="32.1954" width="0" layer="19" extent="1-1"/>
-<wire x1="6.819" y1="31.6992" x2="17.7428" y2="30.5308" width="0" layer="19" extent="1-1"/>
+<wire x1="17.7428" y1="30.5308" x2="21.9202" y2="28.9188" width="0" layer="19" extent="1-1"/>
+<wire x1="26.5338" y1="27.0002" x2="21.9202" y2="28.9188" width="0" layer="19" extent="1-1"/>
+<wire x1="6.8952" y1="29.972" x2="17.7428" y2="30.5308" width="0" layer="19" extent="1-1"/>
 </signal>
 <signal name="N$15">

Commit message: Finished Take 004, Airwire Errors
Parts:
- removed OP4: (no value), LinnesLab-AnalogIC:SOT23-5
- removed U$4: AD5171, LinnesLab-DigitalIC:SOT-23-8
- removed U1: AD5242-SO16, LinnesLab-DigitalIC:SO16
- added AD5171: AD5171, LinnesLab-DigitalIC:SOT-23-8
- added AD5242: AD5242-SO16, LinnesLab-DigitalIC:SO16
- added C2: 100n, LinnesLab-Passives:C0603
- added TIA: (no value), LinnesLab-AnalogIC:SOT23-5
- J1: device LinnesLab-Connectors:1X07 -> LinnesLab-Connectors:1X07_1.27MM
- moved R19 34.0 mm to (32.5, 8.67), turned to 270 degrees
- moved R20 31.4 mm to (29.5, 6.01), turned to 180 degrees
- moved R13 29.1 mm to (33.1, 5.32), turned to 270 degrees
- moved R23 28.5 mm to (29.4, 22.6), turned to 180 degrees
- moved C15 26.5 mm to (29.5, 4.42), turned to 0 degrees
- moved R21 26.1 mm to (31.9, 17.8), turned to 270 degrees
- moved C19 25.1 mm to (29.4, 20.7), turned to 180 degrees
- moved R22 23.5 mm to (29.4, 19.1)
- moved C14 22.2 mm to (29.7, 7.81), turned to 180 degrees
- moved C11 21.8 mm to (25.6, 8.49), turned to 90 degrees
- moved IMU1 21.7 mm to (7.71, 28.2), turned to 90 degrees
- moved R14 19.7 mm to (29.8, 9.49), turned to 0 degrees
- moved R16 19.4 mm to (19.0, 29.5)
- moved C1 17.9 mm to (7.69, 24.1), turned to 0 degrees
- moved C20 17.6 mm to (22.2, 7.00), turned to 270 degrees
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Connections:
- removed net LED: Q1.3
- net 3.3V: now also AD5171.2, AD5171.6, AD5242.5, AD5242.6, J1.4, TIA.5; no longer OP4.5, U$4.2, U$4.6, U1.5, U1.6
- net A6/TIA: now also AD5242.3, J1.6, TIA.1; no longer J1.5, OP4.1, U1.3
- net A7/PPG: now also AD5242.14; no longer U1.14
- net D29/LED.CTRL: now also AD5171.8, J1.5; no longer J1.6, U$4.8
- net G.A1: now also AD5242.2; no longer U1.2
- net G.A2: now also AD5242.16; no longer U1.16
- net G.O1: now also AD5242.1; no longer U1.1
- net G.O2: now also AD5242.13; no longer U1.13
- net G.W2: now also AD5242.15; no longer U1.15
- net GND: now also AD5171.3, AD5242.10, AD5242.11, AD5242.12, AD5242.9, C2.1, J1.3, TIA.2, TIA.3; no longer OP4.2, OP4.3, U$4.3, U1.10, U1.11, U1.12, U1.9
- net LED.C: now also Q1.3
- net N$9: now also AD5171.1, AD5171.7; no longer U$4.1, U$4.7
- net PD.C: now also AD5242.4, TIA.4; no longer OP4.4, U1.4
- net SCL: now also AD5171.4, AD5242.7, J1.2; no longer U$4.4, U1.7
- net SDA: now also AD5171.5, AD5242.8, J1.1; no longer U$4.5, U1.8
- net VREF: now also C2.2
Routing:
- net A6/TIA: track 0.00 -> 66.2 mm, vias 0 -> 4
- net A7/PPG: track 0.00 -> 50.9 mm
- net SDA: track 0.00 -> 37.1 mm
- net VREF: track 0.00 -> 36.9 mm, vias 0 -> 3
- net SCL: track 0.00 -> 36.9 mm, vias 0 -> 2
- net GND: track 0.00 -> 28.7 mm, vias 0 -> 14
- net PD.C: track 0.00 -> 24.0 mm, vias 0 -> 2
- net N$19: track 0.00 -> 22.3 mm
- net N$9: track 0.00 -> 19.5 mm
- net D29/LED.CTRL: track 0.00 -> 17.0 mm, vias 0 -> 2
- net N$13: track 0.00 -> 15.4 mm, vias 0 -> 2
- net G.W2: track 0.00 -> 15.4 mm, vias 0 -> 2
- net N$17: track 0.00 -> 11.1 mm, vias 0 -> 2
- net N$16: track 0.00 -> 10.6 mm
- net N$18: track 0.00 -> 5.85 mm
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- added copper zone on layer 16, net GND

Commit message: Finished Take 006
Parts:
- added C3, C5, C6: 1u, LinnesLab-Passives:C0603
- added C4, C7: 4.7u, LinnesLab-Passives:C0603
- added CHRG: MCP73831, LinnesLab-Power:SOT23-5
- added LDO1: MIC5504, LinnesLab-Power:SOT23-5
- added R11: (no value), LinnesLab-Passives:R0603
- added R12: 100k, LinnesLab-Passives:R0603
- added U4: PCF8523, LinnesLab-Clocks:SO8
- added XTAL3: 32.7680kHz, LinnesLab-Clocks:2-SMD.NOLEAD.2.0MMTO1.2MM
Connections:
- new net D27/CHRG.STATUS: CHRG.1, R12.1
- new net N$1: U4.2
- new net N$2: U4.1, XTAL3.P$2
- new net N$3: CHRG.5, R11.2
- new net VBAT: U4.3
- new net VIN1: C5.2, C7.2, CHRG.4, LDO1.1, LDO1.3, R12.2
- new net VLIPO: C4.1, CHRG.3
- net 3.3V: now also C3.1, C6.1, LDO1.5, U4.8
- net GND: now also C3.2, C4.2, C5.1, C6.2, C7.1, CHRG.2, LDO1.2, R11.1, U4.4
- net SCL: now also U4.6
- net SDA: now also U4.5

Commit message: Almost dont with Take 008
Parts:
- removed C4, C7: 4.7u, LinnesLab-Passives:C0603
- removed C5, C6: 1u, LinnesLab-Passives:C0603
- removed CHRG: MCP73831, LinnesLab-Power:SOT23-5
- removed LDO1: MIC5504, LinnesLab-Power:SOT23-5
- removed R11: (no value), LinnesLab-Passives:R0603
- removed R12: 100k, LinnesLab-Passives:R0603
- moved C3 52.4 mm to (33.5, 32.0), turned to 270 degrees
- moved XTAL3 50.8 mm to (24.4, 32.5), turned to 90 degrees
- moved U4 47.3 mm to (28.9, 31.4)
Connections:
- net A6/TIA renamed A5/TIA
- net A7/PPG renamed A4/PPG
- net D29/LED.CTRL renamed D30/LED.CTRL
- removed net D27/CHRG.STATUS: CHRG.1, R12.1
- removed net N$3: CHRG.5, R11.2
- removed net VIN1: C5.2, C7.2, CHRG.4, LDO1.1, LDO1.3, R12.2
- removed net VLIPO: C4.1, CHRG.3
- net 3.3V: no longer C6.1, LDO1.5
- net GND: no longer C4.2, C5.1, C6.2, C7.1, CHRG.2, LDO1.2, R11.1
Routing:
- net SDA: track 37.1 -> 64.7 mm, vias 0 -> 2
- net SCL: track 36.9 -> 59.6 mm, vias 2 -> 4
- net GND: track 28.7 -> 31.3 mm, vias 14 -> 16
- net A4/PPG: track 50.9 -> 50.3 mm

Commit message: Finished Take 008
Connections:
- net N$1: now also XTAL3.P$1
Routing:
- net N$1: track 0.00 -> 1.97 mm
- net N$2: track 0.00 -> 1.83 mm
Changed lines of the file:
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@@
 <wire x1="22.402803125" y1="18.34895625" x2="21.358859375" y2="19.3929" width="0.1524" layer="1"/>
 <wire x1="21.358859375" y1="19.3929" x2="21.358859375" y2="20.6222625" width="0.1524" layer="1"/>
-<wire x1="24.790396875" y1="24.0538" x2="29.733240625" y2="24.0538" width="0.1524" layer="1"/>
+<wire x1="24.790396875" y1="24.0538" x2="26.990040625" y2="24.0538" width="0.1524" layer="1"/>
+<wire x1="26.990040625" y1="24.0538" x2="29.733240625" y2="24.0538" width="0.1524" layer="1"/>
 <wire x1="29.733240625" y1="24.0538" x2="30.266640625" y2="23.5204" width="0.1524" layer="1"/>
 <wire x1="30.266640625" y1="22.619596875" x2="30.240340625" y2="22.593296875" width="0.1524" layer="1"/>
@@
 <wire x1="24.942803125" y1="13.334996875" x2="24.942803125" y2="11.634159375" width="0.1524" layer="1"/>
 <contactref element="C2" pad="2"/>
-<wire x1="30.240340625" y1="22.593296875" x2="26.9748" y2="24.059778125" width="0" layer="19" extent="1-1"/>
+<wire x1="26.9748" y1="24.059778125" x2="26.9840625" y2="24.059778125" width="0.1524" layer="1"/>
+<wire x1="26.9840625" y1="24.059778125" x2="26.990040625" y2="24.0538" width="0.1524" layer="1"/>
 </signal>
 <signal name="N$9">
@@
 <signal name="N$1">
 <contactref element="U4" pad="2"/>
+<contactref element="XTAL3" pad="P$1"/>
+<wire x1="24.414475" y1="31.673896875" x2="24.75981875" y2="32.019240625" width="0.1524" layer="1"/>
+<wire x1="24.75981875" y1="32.019240625" x2="26.23741875" y2="32.019240625" width="0.1524" layer="1"/>
 </signal>
 <signal name="N$2">
 <contactref element="XTAL3" pad="P$2"/>
 <contactref element="U4" pad="1"/>
-<wire x1="24.414475" y1="33.273896875" x2="26.23741875" y2="33.289240625" width="0" layer="19" extent="1-1"/>
+<wire x1="26.23741875" y1="33.289240625" x2="26.222075" y2="33.273896875" width="0.1524" layer="1"/>
+<wire x1="26.222075" y1="33.273896875" x2="24.414475" y2="33.273896875" width="0.1524" layer="1"/>
 </signal>
 </signals>
