File: Hardware/Bottom/Smarty-BOTTOM.sch (EAGLE design)
At the start: 31 parts, among them U1 AD5242-SO16

Commit message: Finished Take 2
Parts:
- added J1: (no value), LinnesLab-Connectors:CONN_07
Connections:
- removed net LED.CTRL: U$4.A
- removed net PPG: C21.2, OP3G$1.OUT, U1.B2
- removed net TIA: C10.2, C15.1, OP4G$1.OUT, U1.W1
- new net A6/TIA: C10.2, C15.1, J1.5, OP4G$1.OUT, U1.W1
- new net A7/PPG: C21.2, J1.7, OP3G$1.OUT, U1.B2
- new net D29/LED.CTRL: J1.6, U$4.A
Changed lines of the file:
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@@
 <part name="GND2" library="LinnesLab-Symbols" deviceset="GND" device=""/>
 <part name="SUPPLY3" library="LinnesLab-Symbols" deviceset="3.3V" device=""/>
+<part name="J1" library="LinnesLab-Connectors" deviceset="CONN_07" device=""/>
 </parts>
 <sheets>
@@
 <attribute name="VALUE" x="27.94" y="23.114" size="1.778" layer="96" align="bottom-center"/>
 </instance>
+<instance part="J1" gate="G$1" x="106.68" y="0" smashed="yes">
+<attribute name="VALUE" x="101.6" y="-9.906" size="1.778" layer="96" font="vector"/>
+<attribute name="NAME" x="101.6" y="13.208" size="1.778" layer="95" font="vector"/>
+</instance>
 </instances>
 <busses>
@@
 </segment>
 </net>
-<net name="TIA" class="0">
+<net name="A6/TIA" class="0">
 <segment>
 <wire x1="132.08" y1="50.8" x2="127" y2="50.8" width="0.1524" layer="91"/>
@@
 <junction x="81.28" y="129.54"/>
 </segment>
+<segment>
+<pinref part="J1" gate="G$1" pin="5"/>
+<wire x1="111.76" y1="5.08" x2="114.3" y2="5.08" width="0.1524" layer="91"/>
+<label x="114.3" y="5.08" size="1.27" layer="95" xref="yes"/>
+</segment>
 </net>
 <net name="PD.C" class="0">
@@
 </segment>
 </net>
-<net name="LED.CTRL" class="0">
+<net name="D29/LED.CTRL" class="0">
 <segment>
 <pinref part="U$4" gate="G$1" pin="A"/>
@@
 <wire x1="228.6" y1="53.34" x2="228.6" y2="60.96" width="0.1524" layer="91"/>
 <label x="228.6" y="60.96" size="1.27" layer="95" rot="R180" xref="yes"/>
+</segment>
+<segment>
+<pinref part="J1" gate="G$1" pin="6"/>
+<wire x1="111.76" y1="7.62" x2="114.3" y2="7.62" width="0.1524" layer="91"/>
+<label x="114.3" y="7.62" size="1.27" layer="95" xref="yes"/>
 </segment>
 </net>
@@
 </segment>
 </net>
-<net name="PPG" class="0">
+<net name="A7/PPG" class="0">
 <segment>
 <wire x1="160.02" y1="50.8" x2="162.56" y2="50.8" width="0.1524" layer="91"/>
@@
 <label x="220.98" y="121.92" size="1.27" layer="95" xref="yes"/>
 </segment>
-</net>
+<segment>
+<pinref part="J1" gate="G$1" pin="7"/>
+<wire x1="111.76" y1="10.16" x2="114.3" y2="10.16" width="0.1524" layer="91"/>
+<label x="114.3" y="10.16" size="1.27" layer="95" xref="yes"/>
+</segment>
+</net>

Commit message: Finished Take 004, Airwire Errors
Parts:
- removed OP4: (no value), LinnesLab-AnalogIC:OP-SINGLEOT
- added C2: 100n, LinnesLab-Passives:CAPACITOR0603
- added TIA: (no value), LinnesLab-AnalogIC:OP-SINGLEOT
- J1: device LinnesLab-Connectors:CONN_07 -> LinnesLab-Connectors:CONN_07-1.27MM
- renumbered U$4 to AD5171, U1 to AD5242
Connections:
- removed net LED: Q1.C
- net 3.3V: now also J1.4, TIAG$2.V+; no longer OP4G$2.V+
- net A6/TIA: now also J1.6, TIAG$1.OUT; no longer J1.5, OP4G$1.OUT
- net D29/LED.CTRL: now also J1.5; no longer J1.6
- net GND: now also C2.1, J1.3, TIAG$1.+IN, TIAG$2.V-; no longer OP4G$1.+IN, OP4G$2.V-
- net LED.C: now also Q1.C
- net PD.C: now also TIAG$1.-IN; no longer OP4G$1.-IN
- net SCL: now also J1.2
- net SDA: now also J1.1
- net VREF: now also C2.2
Other:
- note added: "Accelerometer and Gyroscope"
- note added: "Castellated IMU Breakout"
- note added: "Connection to Digital Potetiometer for Gain Control"
- note added: "Connection to Optical Sensor Module"
- note added: "Connection to Upper Board"
- note added: "Pins"
- note added: "Vref Generator and Bypass Capacitors"
- moved on the sheet: C1, C10, C11, C14, C15, C16, C19, C20, C21, C22, IMU1, J1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

Commit message: Finished Take 006
Parts:
- added C3, C5, C6: 1u, LinnesLab-Passives:CAPACITOR0603
- added C4, C7: 4.7u, LinnesLab-Passives:CAPACITOR0603
- added CHRG: MCP73831, LinnesLab-Power:MCP73831
- added LDO1: MIC5504, LinnesLab-Power:MIC5504
- added R11: (no value), LinnesLab-Passives:RESISTOR0603
- added R12: 100k, LinnesLab-Passives:RESISTOR0603
- added U4: PCF8523, LinnesLab-Clocks:PCF8523
- added XTAL3: 32.7680kHz, LinnesLab-Clocks:CRYSTALECS-.327-12.5-12-C-TR
Connections:
- new net D27/CHRG.STATUS: CHRG.STAT, R12.1
- new net N$1: U4.OSCO
- new net N$2: U4.OSCI, XTAL3.2
- new net N$3: CHRG.PROG, R11.2
- new net VIN1: C5.2, C7.2, CHRG.VIN, LDO1.EN, LDO1.IN, R12.2
- new net VLIPO: C4.1, CHRG.VBAT
- net 3.3V: now also C3.1, C6.1, LDO1.OUT, U4.VDD
- net GND: now also C3.2, C4.2, C5.1, C6.2, C7.1, CHRG.VSS, LDO1.GND, R11.1, U4.VSS
- net SCL: now also U4.SCL
- net SDA: now also U4.SDA
Other:
- note added: "Digital Output"
- note added: "I2C Address = 0x68h"
- note added: "Real-Time Clock"

Commit message: Almost dont with Take 008
Parts:
- removed C4, C7: 4.7u, LinnesLab-Passives:CAPACITOR0603
- removed C5, C6: 1u, LinnesLab-Passives:CAPACITOR0603
- removed CHRG: MCP73831, LinnesLab-Power:MCP73831
- removed LDO1: MIC5504, LinnesLab-Power:MIC5504
- removed R11: (no value), LinnesLab-Passives:RESISTOR0603
- removed R12: 100k, LinnesLab-Passives:RESISTOR0603
Connections:
- net A6/TIA renamed A5/TIA
- net A7/PPG renamed A4/PPG
- net D29/LED.CTRL renamed D30/LED.CTRL
- removed net D27/CHRG.STATUS: CHRG.STAT, R12.1
- removed net N$3: CHRG.PROG, R11.2
- removed net VIN1: C5.2, C7.2, CHRG.VIN, LDO1.EN, LDO1.IN, R12.2
- removed net VLIPO: C4.1, CHRG.VBAT
- net 3.3V: no longer C6.1, LDO1.OUT
- net GND: no longer C4.2, C5.1, C6.2, C7.1, CHRG.VSS, LDO1.GND, R11.1
Other:
- note added: "Real-Time Clock (RTC)"
- note removed: "Digital Output"
- note removed: "Real-Time Clock"
- moved on the sheet: C3, U4, XTAL3

Commit message: Finished Take 008
Connections:
- net N$1: now also XTAL3.1
Changed lines of the file:
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@@
 <net name="N$1" class="0">
 <segment>
-<wire x1="120.65" y1="-7.62" x2="110.49" y2="-7.62" width="0.1524" layer="91"/>
+<wire x1="120.65" y1="-7.62" x2="111.76" y2="-7.62" width="0.1524" layer="91"/>
 <pinref part="U4" gate="G$1" pin="OSCO"/>
+<pinref part="XTAL3" gate="G$1" pin="1"/>
+<wire x1="111.76" y1="-7.62" x2="110.49" y2="-7.62" width="0.1524" layer="91"/>
+<wire x1="113.03" y1="-5.08" x2="109.22" y2="-5.08" width="0.1524" layer="91"/>
+<wire x1="109.22" y1="-5.08" x2="109.22" y2="-7.62" width="0.1524" layer="91"/>
+<wire x1="109.22" y1="-7.62" x2="110.49" y2="-7.62" width="0.1524" layer="91"/>
 </segment>
 </net>

Commit message: Take 001 Programming 1:09
Other:
- note added: "Gain = -Rf (in pass band)"
- note added: "I_B = (3.3V-0.6V) / (R_pot + R16) LED_current = I_B * Gain Current gain of an NPN transistor is often written as HFE in datasheets"
Changed lines of the file:
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@@
 and LEDs</text>
 <text x="154.94" y="157.48" size="2.54" layer="97" font="vector" ratio="15">Active Bandpass Filters</text>
-<text x="162.56" y="68.58" size="2.54" layer="97" font="vector" ratio="15">Digital Potentiometers</text>
+<text x="162.56" y="76.2" size="2.54" layer="97" font="vector" ratio="15">Digital Potentiometers</text>
 <text x="66.04" y="157.48" size="2.54" layer="97" font="vector" ratio="15">Transimpedance Amplifier</text>
 <text x="134.62" y="27.94" size="1.778" layer="97" ratio="15">I2C Address: 0x2C</text>
@@
 <wire x1="266.7" y1="-33.02" x2="-5.08" y2="-33.02" width="1.016" layer="94"/>
 <wire x1="-5.08" y1="-33.02" x2="-5.08" y2="172.72" width="1.016" layer="94"/>
-<wire x1="0" y1="78.74" x2="45.72" y2="78.74" width="1.016" layer="97" style="longdash"/>
-<wire x1="45.72" y1="78.74" x2="101.6" y2="78.74" width="1.016" layer="97" style="longdash"/>
-<wire x1="101.6" y1="78.74" x2="261.62" y2="78.74" width="1.016" layer="97" style="longdash"/>
-<wire x1="101.6" y1="78.74" x2="101.6" y2="22.86" width="1.016" layer="97" style="longdash"/>
+<wire x1="0" y1="83.82" x2="45.72" y2="83.82" width="1.016" layer="97" style="longdash"/>
+<wire x1="45.72" y1="83.82" x2="101.6" y2="83.82" width="1.016" layer="97" style="longdash"/>
+<wire x1="101.6" y1="83.82" x2="261.62" y2="83.82" width="1.016" layer="97" style="longdash"/>
+<wire x1="101.6" y1="83.82" x2="101.6" y2="22.86" width="1.016" layer="97" style="longdash"/>
 <wire x1="101.6" y1="22.86" x2="101.6" y2="-27.94" width="1.016" layer="97" style="longdash"/>
 <wire x1="101.6" y1="22.86" x2="261.62" y2="22.86" width="1.016" layer="97" style="longdash"/>
 <wire x1="101.6" y1="22.86" x2="60.96" y2="22.86" width="1.016" layer="97" style="longdash"/>
 <wire x1="60.96" y1="22.86" x2="0" y2="22.86" width="1.016" layer="97" style="longdash"/>
-<wire x1="45.72" y1="167.64" x2="45.72" y2="78.74" width="1.016" layer="97" style="longdash"/>
+<wire x1="45.72" y1="167.64" x2="45.72" y2="83.82" width="1.016" layer="97" style="longdash"/>
 <text x="12.7" y="91.44" size="1.778" layer="97">Connection to
 Optical Sensor Module</text>
@@
 <text x="7.62" y="12.7" size="2.54" layer="97" font="vector" ratio="15">Accelerometer and Gyroscope</text>
 <text x="76.2" y="15.24" size="2.54" layer="97" font="vector" ratio="15">Pins</text>
-<text x="22.86" y="71.12" size="2.54" layer="97" font="vector" ratio="15">Vref Generator and Bypass Capacitors</text>
+<text x="22.86" y="76.2" size="2.54" layer="97" font="vector" ratio="15">Vref Generator and Bypass Capacitors</text>
 <text x="143.51" y="-17.78" size="1.27" layer="97">I2C Address = 0x68h</text>
 <text x="115.57" y="8.89" size="4.318" layer="97" font="vector" ratio="15">Real-Time Clock (RTC)</text>
+<text x="218.44" y="66.04" size="1.778" layer="97">I_B = (3.3V-0.6V) / (R_pot + R16)
+LED_current = I_B * Gain
+Current gain of an NPN transistor is
+often written as HFE in datasheets</text>
+<text x="71.12" y="104.14" size="1.778" layer="97">Gain = -Rf (in pass band)</text>
 </plain>
 <instances>
